Commit message: 引入moveit框架

File: src/core/arm_description/urdf/JGarm.urdf (robot description, URDF)
Before this commit: robot JGarm, 7 links, 6 joints
Links:
- removed link link1
- removed link link2
- removed link link3
- removed link link4
- removed link link5
- removed link link6
- added link link_1, mass 0.60157; collision mesh filename=package://arm_description/meshes/link1.STL; visual mesh filename=package://arm_description/meshes/link1.STL
- added link link_2, mass 0.24857; collision mesh filename=package://arm_description/meshes/link2.STL; visual mesh filename=package://arm_description/meshes/link2.STL
- added link link_3, mass 0.89087; collision mesh filename=package://arm_description/meshes/link3.STL; visual mesh filename=package://arm_description/meshes/link3.STL
- added link link_4, mass 0.34032; collision mesh filename=package://arm_description/meshes/link4.STL; visual mesh filename=package://arm_description/meshes/link4.STL
- added link link_5, mass 0.11997; collision mesh filename=package://arm_description/meshes/link5.STL; visual mesh filename=package://arm_description/meshes/link5.STL
- added link link_6, mass 0.56394; collision mesh filename=package://arm_description/meshes/link6.STL; visual mesh filename=package://arm_description/meshes/link6.STL
- link base_link: mass 0.747471424523758 -> None
Joints:
- removed joint joint1
- removed joint joint2
- removed joint joint3
- removed joint joint4
- removed joint joint5
- removed joint joint6
- added joint joint_1: type revolute, parent base_link, child link_1, origin xyz=0 0 0 rpy=0 0 0, axis 0 0 1, limit lower=-3.14 upper=3.14 effort=25 velocity=7.75
- added joint joint_2: type revolute, parent link_1, child link_2, origin xyz=0.03 0.05 0.06 rpy=1.5708 0 -3.1416, axis 0 0 1, limit lower=-1.528 upper=1.084 effort=63 velocity=4.71
- added joint joint_3: type revolute, parent link_2, child link_3, origin xyz=0 0.38 0 rpy=0 0 1.5708, axis 0 0 1, limit lower=-0.5335 upper=1.450 effort=35 velocity=4.71
- added joint joint_4: type revolute, parent link_3, child link_4, origin xyz=-0.005 0.1535 -0.05 rpy=-1.5708 0 0, axis 0 0 1, limit lower=-3.14 upper=3.14 effort=18 velocity=7.54
- added joint joint_5: type revolute, parent link_4, child link_5, origin xyz=0 0 0.136 rpy=1.5708 0.022902 0, axis 0 0 -1, limit lower=-1.967 upper=1.937 effort=6 velocity=20
- added joint joint_6: type revolute, parent link_5, child link_6, origin xyz=0 0.1685 0 rpy=1.5708 0 0, axis 0 0 1, limit lower=-3.14 upper=3.14 effort=3 velocity=10

Commit message: 重构状态机并添加遥控器控制

File: src/core/arm_description/urdf/JGarm.urdf (robot description, URDF)
Before this commit: robot JGarm, 7 links, 6 joints
Joints:
- joint joint_3: limit lower=-0.5335 upper=1.450 effort=35 velocity=4.71 -> lower=-1.2566 upper=1.3972 effort=35 velocity=4.71

Commit message: 重力补偿和摩擦补偿

File: src/core/arm_description/urdf/JGarm.urdf (robot description, URDF)
Before this commit: robot JGarm, 7 links, 6 joints
Joints:
- joint joint_6: axis 0 0 1 -> 0 0 -1

Commit message: 修复部分已知bug

File: src/core/arm_description/urdf/JGarm.urdf (robot description, URDF)
Before this commit: robot JGarm, 7 links, 6 joints
Joints:
- joint joint_2: limit lower=-1.528 upper=1.084 effort=63 velocity=4.71 -> lower=-1.3265 upper=1.9024 effort=63 velocity=4.71
- joint joint_3: limit lower=-1.2566 upper=1.3972 effort=35 velocity=4.71 -> lower=-0.5934 upper=1.3265 effort=35 velocity=4.71
- joint joint_5: origin xyz=0 0 0.136 rpy=1.5708 0.022902 0 -> xyz=0 0 0.136 rpy=1.5708 0 0
